Commit message: Fix Gazebo simulation physics, controllers, and sensor plugins

File: aeroterrabot_ws/src/aeroterrabot_description/urdf/robot.urdf.xacro (robot description, xacro)
@@ -1,4 +1,7 @@
 <?xml version="1.0"?>
 <robot xmlns:xacro="http://www.ros.org/wiki/xacro" name="aeroterrabot">
+    <!-- ── Xacro arguments ─────────────────────────────────────────────── -->
+    <xacro:arg name="use_sim_time" default="false" />
+    <xacro:property name="use_sim" value="$(arg use_sim_time)" />
     <!-- Include the core robot components -->
     <xacro:include filename="robot_core.xacro" />
@@ -7,8 +10,11 @@
     <!-- Include the ros2_control configuration -->
     <xacro:include filename="ros2_control.xacro" />
-    <!-- Example of parameterizing the hardware interface -->
+    <!-- Include the sensors configuration -->
+    <xacro:include filename="sensors.xacro" />
+    <!-- Parameterize the hardware interface -->
     <xacro:aeroterrabot_ros2_control
         serial_port="/dev/ttyACM0"
         baud_rate="115200"
+        use_sim="${use_sim}"
     />
 </robot>

File: aeroterrabot_ws/src/aeroterrabot_description/urdf/robot_core.xacro (robot description, xacro)
@@ -33,4 +33,30 @@
     </xacro:inertial_box>
   </link>
+  <!-- ── LANDING GEAR ────────────────────────────────────────────────────────── -->
+  <xacro:macro name="landing_gear_leg" params="name x y">
+    <joint name="landing_gear_${name}_joint" type="fixed">
+      <parent link="chassis"/>
+      <child link="landing_gear_${name}"/>
+      <origin xyz="${x} ${y} -0.01" rpy="0 0 0"/>
+    </joint>
+    <link name="landing_gear_${name}">
+      <visual>
+        <origin xyz="0 0 0" rpy="0 0 0"/>
+        <geometry><cylinder radius="0.01" length="0.02"/></geometry>
+        <material name="black"/>
+      </visual>
+      <collision>
+        <origin xyz="0 0 0" rpy="0 0 0"/>
+        <geometry><cylinder radius="0.01" length="0.02"/></geometry>
+      </collision>
+      <xacro:inertial_cylinder mass="0.05" length="0.02" radius="0.01">
+        <origin xyz="0 0 0" rpy="0 0 0"/>
+      </xacro:inertial_cylinder>
+    </link>
+  </xacro:macro>
+  <xacro:landing_gear_leg name="front_left" x="0.28" y="0.08" />
+  <xacro:landing_gear_leg name="front_right" x="0.28" y="-0.08" />
+  <xacro:landing_gear_leg name="rear_left" x="0.02" y="0.08" />
+  <xacro:landing_gear_leg name="rear_right" x="0.02" y="-0.08" />
   <!-- ── LEFT MORPHING MECHANISM ────────────────────────────────────────────── -->
   <!-- Actuator pushes left boom outwards. Servo rolls it 90 degrees to point wheels UP. -->
@@ -117,4 +143,10 @@
       <material name="black"/>
     </visual>
+    <!-- Spoke to make rotation visible -->
+    <visual>
+      <origin xyz="0.06 0 0.02" rpy="0 0 0"/>
+      <geometry><box size="0.02 0.02 0.04"/></geometry>
+      <material name="white"/>
+    </visual>
     <collision>
       <geometry><cylinder length="0.03" radius="0.12"/></geometry>
@@ -135,4 +167,10 @@
       <material name="black"/>
     </visual>
+    <!-- Spoke to make rotation visible -->
+    <visual>
+      <origin xyz="0.06 0 0.02" rpy="0 0 0"/>
+      <geometry><box size="0.02 0.02 0.04"/></geometry>
+      <material name="white"/>
+    </visual>
     <collision>
       <geometry><cylinder length="0.03" radius="0.12"/></geometry>
@@ -153,4 +191,10 @@
       <material name="black"/>
     </visual>
+    <!-- Spoke to make rotation visible -->
+    <visual>
+      <origin xyz="0.06 0 0.02" rpy="0 0 0"/>
+      <geometry><box size="0.02 0.02 0.04"/></geometry>
+      <material name="white"/>
+    </visual>
     <collision>
       <geometry><cylinder length="0.03" radius="0.12"/></geometry>
@@ -171,11 +215,34 @@
       <material name="black"/>
     </visual>
-    <collision>
-      <geometry><cylinder length="0.03" radius="0.12"/></geometry>
-    </collision>
-    <xacro:inertial_cylinder mass="0.1" length="0.03" radius="0.12">
-      <origin xyz="0 0 0" rpy="0 0 0"/>
-    </xacro:inertial_cylinder>
-  </link>
+    <!-- Spoke to make rotation visible -->
+    <visual>
+      <origin xyz="0.06 0 0.02" rpy="0 0 0"/>
+      <geometry><box size="0.02 0.02 0.04"/></geometry>
+      <material name="white"/>
+    </visual>
+    <collision>
+      <geometry><cylinder length="0.03" radius="0.12"/></geometry>
+    </collision>
+    <xacro:inertial_cylinder mass="0.1" length="0.03" radius="0.12">
+      <origin xyz="0 0 0" rpy="0 0 0"/>
+    </xacro:inertial_cylinder>
+  </link>
+  <!-- Gazebo Friction tags for wheels -->
+  <gazebo reference="front_left_wheel">
+    <mu1>1.0</mu1>
+    <mu2>1.0</mu2>
+  </gazebo>
+  <gazebo reference="front_right_wheel">
+    <mu1>1.0</mu1>
+    <mu2>1.0</mu2>
+  </gazebo>
+  <gazebo reference="rear_left_wheel">
+    <mu1>1.0</mu1>
+    <mu2>1.0</mu2>
+  </gazebo>
+  <gazebo reference="rear_right_wheel">
+    <mu1>1.0</mu1>
+    <mu2>1.0</mu2>
+  </gazebo>
   <!-- ── ROTORS ────────────────────────────────────────────────────────────── -->
   <!-- Rotors attach directly to the boom frame, avoiding rotation when driving -->

File: aeroterrabot_ws/src/aeroterrabot_description/urdf/ros2_control.xacro (robot description, xacro)
@@ -4,13 +4,19 @@
   Include this XACRO in the main robot URDF to register the Teensy 4.0
   SystemInterface plugin with the controller manager.
+  Use use_sim:=true when launching with Gazebo.
 -->
 <robot xmlns:xacro="http://www.ros.org/wiki/xacro">
   <xacro:macro name="aeroterrabot_ros2_control"
-               params="serial_port:=/dev/ttyACM0 baud_rate:=115200">
+               params="serial_port:=/dev/ttyACM0 baud_rate:=115200 use_sim:=false">
     <ros2_control name="AeroTerraBotSystem" type="system">
       <hardware>
-        <plugin>aeroterrabot_hardware/AeroTerraBotSystemInterface</plugin>
-        <param name="serial_port">${serial_port}</param>
-        <param name="baud_rate">${baud_rate}</param>
+        <xacro:if value="${use_sim}">
+          <plugin>gz_ros2_control/GazeboSimSystem</plugin>
+        </xacro:if>
+        <xacro:unless value="${use_sim}">
+          <plugin>aeroterrabot_hardware/AeroTerraBotSystemInterface</plugin>
+          <param name="serial_port">${serial_port}</param>
+          <param name="baud_rate">${baud_rate}</param>
+        </xacro:unless>
       </hardware>
       <!-- ═══ Wheel Joints (velocity) ═══════════════════════════════════ -->
@@ -115,4 +121,13 @@
       </joint>
     </ros2_control>
+    <!-- ── Gazebo Sim Controller Plugin (only active in simulation) ──────── -->
+    <xacro:if value="${use_sim}">
+      <gazebo>
+        <plugin filename="gz_ros2_control-system"
+                name="gz_ros2_control::GazeboSimROS2ControlPlugin">
+          <parameters>$(find aeroterrabot_control)/config/controllers.yaml</parameters>
+        </plugin>
+      </gazebo>
+    </xacro:if>
   </xacro:macro>
 </robot>
